File: temp_fan_node/temp_fan_node.kicad_pcb (KiCad board)
At the start: 2 copper layers, 50.8 x 38.1 mm, 40 parts, among them J1 temp_1, J2 temp_2, J3 temp_3, J4 PWR_in, J5 SW_Fan_GND, J6 rs-485, J7 temp_4, J8 O2_sensor, Q1 IRLS3036, U1 ATtiny3216-S, U2 AP63205WU, U3 AP2112K-3.3, U4 MCP1406-E/SN, U5 THVD1420D

Commit message: Add alternator 555 timer and ESP32 UPDI programmer to monorepo.
Consolidate T-Bird hardware projects under smart_tbird and update temp_fan_node KiCad files.

Co-authored-by: Cursor <cursoragent@cursor.com>
Parts:
- added C10: 0.1uF, Capacitor_SMD:C_1206_3216Metric_Pad1.33x1.80mm_HandSolder, F.Cu at (79.4, 62.0)
- added C11: 0.1uF, Capacitor_SMD:C_1206_3216Metric_Pad1.33x1.80mm_HandSolder, F.Cu at (82.4, 65.0)
- added C12: 0.1uF, Capacitor_SMD:C_1206_3216Metric_Pad1.33x1.80mm_HandSolder, F.Cu at (76.4, 65.0)
- added C13: 0.1uF, Capacitor_SMD:C_1206_3216Metric_Pad1.33x1.80mm_HandSolder, F.Cu at (84.4, 45.0)
- added C14: 0.1uF, Capacitor_SMD:C_1206_3216Metric_Pad1.33x1.80mm_HandSolder, F.Cu at (76.4, 45.0)
- added C15: 0.1uF, Capacitor_SMD:C_1206_3216Metric_Pad1.33x1.80mm_HandSolder, F.Cu at (100.0, 64.6)
- added C9: 0.1uF, Capacitor_SMD:C_1206_3216Metric_Pad1.33x1.80mm_HandSolder, F.Cu at (85.4, 62.0)
- added J9: GND_conn, Connector:Alex_1pin_065thou, F.Cu at (82.0, 73.0)
- added R12: 120, Resistor_SMD:R_1206_3216Metric_Pad1.30x1.75mm_HandSolder, F.Cu at (99.0, 69.7)
- moved C4 12.7 mm to (95.4, 56.0), turned to 180 degrees
- moved J3 7.09 mm to (83.0, 69.0)
- moved J1 7.07 mm to (77.0, 69.0)
- moved R7 7.02 mm to (86.0, 63.5)
- moved R2 5.73 mm to (83.0, 63.4), turned to -90 degrees
- moved U3 5.18 mm to (99.5, 61.9)
- moved J7 4.58 mm to (86.0, 69.0)
- moved R8 3.00 mm to (88.0, 42.0)
- moved TH1 3.00 mm to (82.4, 42.0)
- moved J2 2.83 mm to (80.0, 69.0)
- moved Q1 2.55 mm to (111.5, 51.1)
- moved C6 2.12 mm to (101.6, 56.0), turned to 180 degrees
- moved R1 1.69 mm to (80.0, 63.4), turned to -90 degrees
- moved J6 1.53 mm to (97.5, 74.0), turned to 0 degrees
- moved U5 1.14 mm to (92.1, 66.1)
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Connections:
- F1 pad 2: GND -> Net-(J4-Pin_2)
- J4 pad 2: /12V -> Net-(J4-Pin_2)
- R4 pad 1: /12V -> Net-(J4-Pin_2)
- R6 pad 2: /12V -> Net-(J4-Pin_2)
- U4 pad 1: /12V -> Net-(J4-Pin_2)
- U4 pad 8: /12V -> Net-(J4-Pin_2)
Routing:
- net Net-(U1-PA3): track 1.27 -> 0.00 mm
- net Net-(J1-Pin_1): track 1.02 -> 0.00 mm
- net Net-(U1-PA2): track 0.97 -> 0.00 mm
- net GND: track 0.54 -> 0.00 mm
Other:
- board text added: "A"
- board text added: "B"
