File: temp_fan_node/temp_fan_node.kicad_sch (KiCad schematic)
At the start: 40 parts, among them J1 temp_1, J2 temp_2, J3 temp_3, J4 PWR_in, J5 SW_Fan_GND, J6 rs-485, J7 temp_4, J8 O2_sensor, Q1 IRLS3036, U1 ATtiny3216-S, U2 AP63205WU, U3 AP2112K-3.3, U4 MCP1406-E/SN, U5 THVD1420D

Commit message: Add alternator 555 timer and ESP32 UPDI programmer to monorepo.
Consolidate T-Bird hardware projects under smart_tbird and update temp_fan_node KiCad files.

Co-authored-by: Cursor <cursoragent@cursor.com>
Parts:
- added C10, C11, C12, C13, C14, C15, C9: 0.1uF, Capacitor_SMD:C_1206_3216Metric_Pad1.33x1.80mm_HandSolder, symbol Device:C_Small_US
- added J9: GND_conn, Connector:Alex_1pin_065thou, symbol Connector:Conn_01x01_Socket
- added R12: 120, Resistor_SMD:R_1206_3216Metric_Pad1.30x1.75mm_HandSolder, symbol Device:R_Small_US
Connections:
- net 12V: no longer J4.2 (Pin_2), R4.1, R6.2, U4.1 (VDD), U4.8 (VDD)
- net GND: now also C10.1, C11.1, C12.1, C13.1, C14.1, C15.1, C9.1, J9.1 (Pin_1); no longer F1.2
- net at D2.2 (A2), J6.1 (Pin_1), U5.6 (A): now also R12.2
- net at D2.1 (A1), J6.2 (Pin_2), U5.7 (B): now also R12.1
- net at J3.1 (Pin_1), R3.2, U1.13 (PC1): now also C10.2
- net at R5.1, R6.1, U1.10 (PB1): now also C14.2
- net at J1.1 (Pin_1), R1.2, U1.12 (PC0): now also C12.2
- net at J2.1 (Pin_1), R2.2, U1.14 (PC2): now also C11.2
- net at J7.1 (Pin_1), R7.2, U1.15 (PC3): now also C9.2
- net at R8.1, TH1.1, U1.3 (PA5): now also C13.2
- net at R11.1, R9.2, U1.8 (PB3): now also C15.2
- new net: F1.2, J4.2 (Pin_2), R4.1, R6.2, U4.1 (VDD), U4.8 (VDD)
Other:
- note added: "5V max from O2 sensor"
- note added: "O2 GND"
- moved on the sheet: F1, J4, J6, R11, R9
