File: alternator_555_timer/alternator_555_timer.kicad_sch (KiCad schematic)
At the start: 18 parts, among them J1 I_In, J2 I_out, J3 GND_Conn, Q1 FQD11P06TM, U1 TLC555CP

Commit message: project progress
Parts:
- D3: value Green LED -> G. LED
- D4: value Red LED -> R. LED
- J1, J2, J3: footprint Connector_Pin:12_AWG_TH_Alex -> Connector:Alex_1pin_065thou
Connections:
- net at D1.1 (K), D4.2 (A), J2.1 (Pin_1): now also Q1.2 (D); no longer Q1.3 (S)
- net at D3.2 (A): now also Q1.3 (S); no longer Q1.2 (D)
Changed lines of the file:
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@@
+	)
+	(junction
+		(at 182.88 93.98)
+		(diameter 0)
+		(color 0 0 0 0)
 	)
 	(junction
 		(at 168.91 93.98)
-		(diameter 0)
-		(color 0 0 0 0)
-	)
-	(junction
-		(at 182.88 93.98)
 		(diameter 0)
 		(color 0 0 0 0)
@@
 			)
 		)
-		(property "Value" "Red LED"
+		(property "Value" "R. LED"
 			(at 195.8975 113.03 0)
 			(show_name no)
@@
 			)
 		)
-		(property "Footprint" "Connector_Pin:12_AWG_TH_Alex"
+		(property "Footprint" "Connector:Alex_1pin_065thou"
 			(at 71.12 78.74 0)
 			(hide yes)
@@
 			)
 		)
-		(property "Value" "Green LED"
+		(property "Value" "G. LED"
 			(at 195.8975 66.04 0)
 			(show_name no)
@@
 			)
 		)
-		(property "Footprint" "Connector_Pin:12_AWG_TH_Alex"
+		(property "Footprint" "Connector:Alex_1pin_065thou"
 			(at 130.81 113.03 0)
 			(hide yes)
@@
 		(lib_id "Transistor_FET:FQP27P06")
 		(at 187.96 93.98 0)
+		(mirror x)
 		(unit 1)
 		(body_style 1)
@@
 		(in_pos_files yes)
 		(dnp no)
-		(fields_autoplaced yes)
 		(property "Reference" "Q1"
 			(at 194.31 92.7099 0)
@@
 		)
 		(property "Footprint" "Package_TO_SOT_SMD:TO-252-2"
-			(at 193.04 95.885 0)
+			(at 193.04 92.075 0)
 			(hide yes)
 			(show_name no)
@@
 		)
 		(property "Datasheet" "https://www.onsemi.com/pub/Collateral/FQP27P06-D.PDF"
-			(at 193.04 97.79 0)
+			(at 193.04 90.17 0)
 			(hide yes)
 			(show_name no)
@@
 			)
 		)
-		(property "Footprint" "Connector_Pin:12_AWG_TH_Alex"
+		(property "Footprint" "Connector:Alex_1pin_065thou"
 			(at 195.58 104.14 0)
 			(hide yes)
