File: alternator_555_timer/alternator_555_timer.kicad_sch (KiCad schematic)
At the start: 18 parts, among them J1 I_In, J2 I_out, J3 GND_Conn, Q1 FQD11P06TM, U1 TLC555CP

Commit message: PCB Updates
Connections:
- net at D4.2 (A), J2.1 (Pin_1), Q1.2 (D): no longer D1.1 (K)
- net at D3.2 (A), Q1.3 (S): now also D1.1 (K)
Other:
- moved on the sheet: D1
Changed lines of the file:
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@@
+	)
+	(junction
+		(at 179.07 93.98)
+		(diameter 0)
+		(color 0 0 0 0)
 	)
 	(junction
@@
 	)
 	(junction
-		(at 182.88 93.98)
+		(at 190.5 77.47)
 		(diameter 0)
 		(color 0 0 0 0)
@@
 	(wire
 		(pts
+			(xy 179.07 93.98) (xy 182.88 93.98)
+		)
+		(stroke
+			(width 0)
+			(type default)
+		)
+	)
+	(wire
+		(pts
 			(xy 115.57 88.9) (xy 115.57 52.07)
 		)
@@
 	(wire
 		(pts
-			(xy 182.88 120.65) (xy 182.88 115.57)
-		)
-		(stroke
-			(width 0)
-			(type default)
-		)
-	)
-	(wire
-		(pts
 			(xy 190.5 99.06) (xy 190.5 104.14)
 		)
@@
 	(wire
 		(pts
+			(xy 190.5 77.47) (xy 190.5 88.9)
+		)
+		(stroke
+			(width 0)
+			(type default)
+		)
+	)
+	(wire
+		(pts
 			(xy 198.12 71.12) (xy 200.66 71.12)
 		)
@@
 	(wire
 		(pts
-			(xy 182.88 93.98) (xy 182.88 107.95)
-		)
-		(stroke
-			(width 0)
-			(type default)
-		)
-	)
-	(wire
-		(pts
 			(xy 153.67 93.98) (xy 168.91 93.98)
 		)
@@
 	(wire
 		(pts
+			(xy 179.07 81.28) (xy 179.07 77.47)
+		)
+		(stroke
+			(width 0)
+			(type default)
+		)
+	)
+	(wire
+		(pts
 			(xy 200.66 118.11) (xy 200.66 120.65)
 		)
@@
 	(wire
 		(pts
-			(xy 168.91 93.98) (xy 182.88 93.98)
+			(xy 168.91 93.98) (xy 179.07 93.98)
 		)
 		(stroke
@@
 	(wire
 		(pts
+			(xy 179.07 88.9) (xy 179.07 93.98)
+		)
+		(stroke
+			(width 0)
+			(type default)
+		)
+	)
+	(wire
+		(pts
 			(xy 77.47 49.53) (xy 95.25 49.53)
 		)
@@
 	(wire
 		(pts
-			(xy 182.88 120.65) (xy 190.5 120.65)
-		)
-		(stroke
-			(width 0)
-			(type default)
-		)
-	)
-	(wire
-		(pts
-			(xy 190.5 71.12) (xy 190.5 88.9)
+			(xy 190.5 71.12) (xy 190.5 77.47)
 		)
 		(stroke
@@
 		(pts
 			(xy 168.91 106.68) (xy 168.91 113.03)
+		)
+		(stroke
+			(width 0)
+			(type default)
+		)
+	)
+	(wire
+		(pts
+			(xy 179.07 77.47) (xy 190.5 77.47)
 		)
 		(stroke
@@
 		)
 		(instances
-			(project "555_I_delay"
+			(project "alternator_555_timer"
 				(path "/686101b5-5487-4618-9623-99f46b13644e"
 					(reference "C1")
@@
 		)
 		(instances
-			(project "555_I_delay"
+			(project "alternator_555_timer"
 				(path "/686101b5-5487-4618-9623-99f46b13644e"
 					(reference "#PWR010")
@@
 		)
 		(instances
-			(project "555_I_delay"
+			(project "alternator_555_timer"
 				(path "/686101b5-5487-4618-9623-99f46b13644e"
 					(reference "#PWR08")
@@
 		)
 		(instances
-			(project "555_I_delay"
+			(project "alternator_555_timer"
 				(path "/686101b5-5487-4618-9623-99f46b13644e"
 					(reference "#PWR07")
@@
 		)
 		(instances
-			(project "555_I_delay"
+			(project "alternator_555_timer"
 				(path "/686101b5-5487-4618-9623-99f46b13644e"
 					(reference "#PWR02")
@@
 		)
 		(instances
-			(project "555_I_delay"
+			(project "alternator_555_timer"
 				(path "/686101b5-5487-4618-9623-99f46b13644e"
 					(reference "C3")
@@
 		)
 		(instances
-			(project "555_I_delay"
+			(project "alternator_555_timer"
 				(path "/686101b5-5487-4618-9623-99f46b13644e"
 					(reference "C4")
@@
 	(symbol
 		(lib_id "Diode:SS33")
-		(at 182.88 111.76 90)
+		(at 179.07 85.09 270)
 		(unit 1)
 		(body_style 1)
@@
 		(fields_autoplaced yes)
 		(property "Reference" "D1"
-			(at 185.42 110.8074 90)
+			(at 181.61 84.7724 90)
+			(show_name no)
+			(do_not_autoplace no)
+			(effects
+				(font
+					(size 1.27 1.27)
+				)
+				(justify left)
+			)
+		)
+		(property "Value" "SZ1SMB15AT3G"
+			(at 176.53 83.5026 90)
+			(hide yes)
 			(show_name no)
 			(do_not_autoplace no)
@@
 			)
 		)
-		(property "Value" "SZ1SMB15AT3G"
-			(at 185.42 113.3474 90)
-			(hide yes)
-			(show_name no)
-			(do_not_autoplace no)
-			(effects
-				(font
-					(size 1.27 1.27)
-				)
-				(justify right)
-			)
-		)
 		(property "Footprint" "Diode_SMD:D_SMB_Handsoldering"
-			(at 187.325 111.76 0)
+			(at 174.625 85.09 0)
 			(hide yes)
 			(show_name no)
@@
 		)
 		(property "Datasheet" ""
-			(at 182.88 111.76 0)
+			(at 179.07 85.09 0)
 			(hide yes)
 			(show_name no)
@@
 		)
 		(property "Description" "Gate/Drain TVS protection"
-			(at 182.88 111.76 0)
+			(at 179.07 85.09 0)
 			(hide yes)
 			(show_name no)
@@
 		)
 		(instances
-			(project "555_I_delay"
+			(project "alternator_555_timer"
 				(path "/686101b5-5487-4618-9623-99f46b13644e"
 					(reference "D1")
@@
 		)
 		(instances
-			(project "555_I_delay"
+			(project "alternator_555_timer"
 				(path "/686101b5-5487-4618-9623-99f46b13644e"
 					(reference "D4")
@@
 		)
 		(instances
-			(project "555_I_delay"
+			(project "alternator_555_timer"
 				(path "/686101b5-5487-4618-9623-99f46b13644e"
 					(reference "#PWR04")
@@
 		)
 		(instances
-			(project "555_I_delay"
+			(project "alternator_555_timer"
 				(path "/686101b5-5487-4618-9623-99f46b13644e"
 					(reference "J1")
@@
 		)
 		(instances
-			(project "555_I_delay"
+			(project "alternator_555_timer"
 				(path "/686101b5-5487-4618-9623-99f46b13644e"
 					(reference "R1")
@@
 		)
 		(instances
-			(project "555_I_delay"
+			(project "alternator_555_timer"
 				(path "/686101b5-5487-4618-9623-99f46b13644e"
 					(reference "#PWR01")
@@
 		)
 		(instances
-			(project "555_I_delay"
+			(project "alternator_555_timer"
 				(path "/686101b5-5487-4618-9623-99f46b13644e"
 					(reference "#PWR09")
@@
 		)
 		(instances
-			(project "555_I_delay"
+			(project "alternator_555_timer"
 				(path "/686101b5-5487-4618-9623-99f46b13644e"
 					(reference "D3")
@@
 		)
 		(instances
-			(project "555_I_delay"
+			(project "alternator_555_timer"
 				(path "/686101b5-5487-4618-9623-99f46b13644e"
 					(reference "R3")
@@
 		)
 		(instances
-			(project "555_I_delay"
+			(project "alternator_555_timer"
 				(path "/686101b5-5487-4618-9623-99f46b13644e"
 					(reference "D2")
@@
 		)
 		(instances
-			(project "555_I_delay"
+			(project "alternator_555_timer"
 				(path "/686101b5-5487-4618-9623-99f46b13644e"
 					(reference "C2")
@@
 		)
 		(instances
-			(project "555_I_delay"
+			(project "alternator_555_timer"
 				(path "/686101b5-5487-4618-9623-99f46b13644e"
 					(reference "J3")
@@
 		)
 		(instances
-			(project "555_I_delay"
+			(project "alternator_555_timer"
 				(path "/686101b5-5487-4618-9623-99f46b13644e"
 					(reference "U1")
@@
 		)
 		(instances
-			(project "555_I_delay"
+			(project "alternator_555_timer"
 				(path "/686101b5-5487-4618-9623-99f46b13644e"
 					(reference "#PWR03")
@@
 		)
 		(instances
-			(project "555_I_delay"
+			(project "alternator_555_timer"
 				(path "/686101b5-5487-4618-9623-99f46b13644e"
 					(reference "Q1")
@@
 		)
 		(instances
-			(project "555_I_delay"
+			(project "alternator_555_timer"
 				(path "/686101b5-5487-4618-9623-99f46b13644e"
 					(reference "R4")
@@
 		)
 		(instances
-			(project "555_I_delay"
+			(project "alternator_555_timer"
 				(path "/686101b5-5487-4618-9623-99f46b13644e"
 					(reference "#PWR06")
@@
 		)
 		(instances
-			(project "555_I_delay"
+			(project "alternator_555_timer"
 				(path "/686101b5-5487-4618-9623-99f46b13644e"
 					(reference "F1")
@@
 		)
 		(instances
-			(project "555_I_delay"
+			(project "alternator_555_timer"
 				(path "/686101b5-5487-4618-9623-99f46b13644e"
 					(reference "R2")
@@
 		)
 		(instances
-			(project "555_I_delay"
+			(project "alternator_555_timer"
 				(path "/686101b5-5487-4618-9623-99f46b13644e"
 					(reference "J2")
