File: engine_monitor/engine_monitor_PCB/engine_monitor.kicad_pcb (KiCad board)
At the start: 2 copper layers, 50.8 x 38.1 mm, 49 parts, among them J1 temp_1, J2 temp_2, J3 temp_3, J4 PWR_in, J5 SW_Fan_GND, J6 rs-485, J7 temp_4, J8 O2_sensor, J9 GND_conn, Q1 IRLS3036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

Commit message: project progress
Parts:
- added C16: 0.1uF, Capacitor_SMD:C_1206_3216Metric_Pad1.33x1.80mm_HandSolder, B.Cu at (76.4, 58.0)
- added C17: 220pF, Capacitor_SMD:C_1206_3216Metric_Pad1.33x1.80mm_HandSolder, B.Cu at (80.2, 50.4)
- added D3: 1N5819, Diode_SMD:D_SOD-123, B.Cu at (85.2, 50.8)
- added D4: 1N5819, Diode_SMD:D_SOD-123, B.Cu at (85.2, 45.2)
- added J10: Tach+, Connector:Alex_1pin_065thou, F.Cu at (76.0, 46.9)
- added J11: Tach-, Connector:Alex_1pin_065thou, F.Cu at (76.0, 52.4)
- added R13: 100k, Resistor_SMD:R_1206_3216Metric_Pad1.30x1.75mm_HandSolder, B.Cu at (80.7, 45.2)
- added R14: 100k, Resistor_SMD:R_1206_3216Metric_Pad1.30x1.75mm_HandSolder, F.Cu at (76.7, 55.2)
- added R15: 6.8k, Resistor_SMD:R_1206_3216Metric_Pad1.30x1.75mm_HandSolder, F.Cu at (81.8, 55.2)
- added R16: 330k, Resistor_SMD:R_1206_3216Metric_Pad1.30x1.75mm_HandSolder, F.Cu at (83.2, 59.5)
- added TP1: 3.3V, TestPoint:TestPoint_Pad_2.5x2.5mm, B.Cu at (99.8, 46.8)
- added TP2: 5V, TestPoint:TestPoint_Pad_2.5x2.5mm, B.Cu at (116.6, 48.4)
- added TP3: UPDI, TestPoint:TestPoint_Pad_2.5x2.5mm, B.Cu at (90.6, 66.6)
- added U6: MCP6561x-LT, Package_TO_SOT_SMD:SOT-23-5, F.Cu at (77.1, 60.2)
- C6, C7: value 1uF -> 4.7uF
- moved R4 15.0 mm to (108.7, 60.4), turned to 0 degrees
- moved F1 9.62 mm to (106.0, 70.9), turned to 0 degrees
- moved C8 8.13 mm to (115.4, 60.4)
- moved U1 8.13 mm to (91.4, 53.2)
- moved C14 6.60 mm to (83.0, 45.2)
- moved D10 4.80 mm to (95.0, 41.2)
- moved C13 4.60 mm to (89.0, 45.2)
- moved R9 4.60 mm to (115.5, 67.6)
- moved R37 4.44 mm to (99.7, 41.2)
- moved C11 3.65 mm to (83.0, 68.6)
- moved C12 3.62 mm to (76.8, 68.6)
- moved J9 3.49 mm to (85.2, 74.4)
- moved J7 3.12 mm to (88.4, 71.0)
- moved R1 2.91 mm to (80.2, 66.2)
- moved C15 2.88 mm to (97.6, 63.0)
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Connections:
- J8 pad 3: /12V -> Net-(J4-Pin_2)
- R4 pad 1: Net-(J4-Pin_2) -> /12V
- R6 pad 2: Net-(J4-Pin_2) -> /12V
- U1 pad 16: unconnected-(U1-~{RESET}/PA0-Pad16) -> Net-(U1-~{RESET}/PA0)
- U1 pad 6: unconnected-(U1-PB5-Pad6) -> Net-(U1-PB5)
- U4 pad 1: Net-(J4-Pin_2) -> /12V
- U4 pad 8: Net-(J4-Pin_2) -> /12V
Routing:
- net Net-(Q1-G): track 0.00 -> 0.70 mm
Other:
- board text added: "FAN PWM"
- board text added: "GND"
- board text added: "In+"
- board text added: "T1"
- board text added: "T2"
- board text added: "T3"
- board text added: "T4"
- board text added: "Tach+"
- board text added: "Tach-"

Commit message: layout for the day
Parts:
- C8: moved to B.Cu
- moved R3 6.40 mm to (80.2, 66.3)
- moved C8 5.86 mm to (114.6, 54.6)
- moved R37 4.44 mm to (100.2, 45.6)
- moved J2 4.00 mm to (84.8, 71.0)
- moved R1 3.80 mm to (76.4, 66.2)
- moved J3 3.60 mm to (81.0, 71.0)
- moved J6 2.34 mm to (99.8, 74.0), turned to 180 degrees
- moved J9 2.28 mm to (83.0, 73.8)
- moved TP3 2.24 mm to (92.8, 66.2)
- moved J5 2.04 mm to (121.4, 48.0)
- moved R16 1.40 mm to (81.8, 59.6)
- moved R10 1.40 mm to (101.8, 49.5)
- moved R7 1.00 mm to (87.6, 66.3)
- moved TP2 1.00 mm to (116.0, 47.6)
- moved D10 0.77 mm to (95.4, 41.9), turned to -90 degrees
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Connections:
- R16 pad 1: Net-(U1-PB5) -> Net-(U1-PB2)
- U1 pad 6: Net-(U1-PB5) -> unconnected-(U1-PB5-Pad6)
- U1 pad 9: unconnected-(U1-PB2-Pad9) -> Net-(U1-PB2)
- U6 pad 1: Net-(U1-PB5) -> Net-(U1-PB2)
Routing:
- net /3.3V: track 0.00 -> 92.9 mm, vias 0 -> 4
- net /12V: track 0.00 -> 56.2 mm
- net /5.5V: track 0.00 -> 43.8 mm
- net Net-(U1-PB1): track 0.00 -> 33.6 mm, vias 0 -> 1
- net Net-(D2-A2): track 0.00 -> 27.1 mm, vias 0 -> 2
- net Net-(D3-A): track 0.00 -> 26.5 mm, vias 0 -> 1
- net Net-(U1-PB3): track 0.00 -> 24.0 mm
- net Net-(J4-Pin_2): track 0.00 -> 22.5 mm
- net Net-(J1-Pin_1): track 0.00 -> 21.5 mm
- net Net-(J3-Pin_1): track 0.00 -> 20.4 mm
- net Net-(J2-Pin_1): track 0.00 -> 18.9 mm
- net Net-(U1-PB2): track 0.00 -> 18.4 mm
- net Net-(J7-Pin_1): track 0.00 -> 18.2 mm
- net Net-(U1-PA4): track 0.00 -> 16.8 mm, vias 0 -> 2
- net Net-(D2-A1): track 0.00 -> 14.5 mm
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Other:
- board text added: "3.3V"
- board text added: "5.0V"
- board text added: "UPDI"

Commit message: PCB updates
Parts:
- removed J11: Tach-, Connector:Alex_1pin_065thou
- added TP4: Tach, Connector:Alex_35thou_wire_hole, F.Cu at (76.2, 52.4)
- moved R9 4.10 mm to (115.5, 63.5)
- moved Q1 3.81 mm to (111.7, 47.4), turned to 90 degrees
- moved R11 3.50 mm to (115.5, 60.5)
- moved F1 1.60 mm to (106.0, 69.3)
- moved D1 1.12 mm to (107.8, 65.0)
- turned R4 to 180 degrees
Connections:
- Q1 pad 1: Net-(J5-Pin_1) -> Net-(Q1-G)
- Q1 pad 2: Net-(Q1-G) -> Net-(J5-Pin_1)
Routing:
- net Net-(U1-PB3): track 24.0 -> 41.9 mm
- net /12V: track 56.2 -> 70.4 mm, vias 0 -> 2
- net Net-(J5-Pin_1): track 9.18 -> 19.7 mm
- net Net-(Q1-G): track 8.97 -> 17.7 mm
- net Net-(D3-A): track 26.5 -> 31.9 mm
- net Net-(J8-Pin_2): track 7.71 -> 5.42 mm
- net Net-(J4-Pin_2): track 22.5 -> 21.6 mm
- net GND: vias 0 -> 14
- added copper zone on B.Cu, net GND
- added copper zone on F.Cu, net GND
Other:
- outline, holes or cut-outs redrawn
- board text added: "O2"
- board text added: "Tach TP"
- board text removed: "Tach-"
