File: engine_monitor/engine_monitor_PCB/engine_monitor.kicad_pcb (KiCad board)
At the start: 2 copper layers, 50.8 x 38.1 mm, 63 parts, among them J1 temp_1, J10 Tach+, J2 temp_2, J3 temp_3, J4 PWR_in, J5 SW_Fan_GND, J6 rs-485, J7 temp_4, J8 O2_sensor, J9 GND_conn, Q1 IRLS3036, U1 ATtiny3216-S, U2 AP63205WU, U3 AP2112K-3.3, U4 MCP1406-E/SN, U5 THVD1420D, U6 MCP6561x-LT

Commit message: checkpoint
Parts:
- R14: value 100k -> 10k
- R15: value 6.8k -> 2k
- R16: value 330k -> 100k
- R8, TH1: moved to B.Cu
- U3: value AP2112K-3.3 -> AP2115M-3.3TRG1
- moved TH1 27.8 mm to (109.8, 45.0), turned to -90 degrees
- moved R8 18.7 mm to (106.2, 45.0), turned to -90 degrees
- moved R5 6.72 mm to (115.2, 40.8)
- moved C8 5.65 mm to (114.6, 60.2)
- moved R6 4.23 mm to (115.2, 43.5)
Connections:
- C15 pad 2: Net-(U1-PB3) -> Net-(U1-PA6)
- R11 pad 1: Net-(U1-PB3) -> Net-(U1-PA6)
- R16 pad 1: Net-(U1-PB2) -> Net-(U1-PB4)
- R9 pad 2: Net-(U1-PB3) -> Net-(U1-PA6)
- U1 pad 4: unconnected-(U1-PA6-Pad4) -> Net-(U1-PA6)
- U1 pad 7: unconnected-(U1-PB4-Pad7) -> Net-(U1-PB4)
- U1 pad 8: Net-(U1-PB3) -> unconnected-(U1-PB3-Pad8)
- U1 pad 9: Net-(U1-PB2) -> unconnected-(U1-PB2-Pad9)
- U6 pad 1: Net-(U1-PB2) -> Net-(U1-PB4)
Routing:
- net Net-(U1-PB3): track 41.9 -> 0.00 mm
- net Net-(U1-PA6): track 0.00 -> 38.3 mm
- net Net-(U1-PB4): track 0.00 -> 19.4 mm
- net Net-(U1-PB2): track 18.4 -> 0.00 mm
- net Net-(U1-PA5): track 14.4 -> 26.6 mm, vias 0 -> 1
- net Net-(J5-Pin_1): track 19.7 -> 10.5 mm
- net /12V: track 70.4 -> 62.5 mm, vias 2 -> 3
- net GND: track 0.00 -> 4.30 mm, vias 14 -> 38
- net Net-(U1-PB1): track 33.6 -> 37.5 mm
- net Net-(J1-Pin_1): track 21.5 -> 22.8 mm
- net Net-(Q1-G): track 17.7 -> 16.7 mm
- net unconnected-(U1-PB3-Pad8): track 0.00 -> 0.70 mm
- net /3.3V: track 92.9 -> 92.3 mm
Other:
- board text added: "SGNL"
