File: engine_monitor/engine_monitor_PCB/engine_monitor.kicad_sch (KiCad schematic)
At the start: 63 parts, among them J1 temp_1, J10 Tach+, J2 temp_2, J3 temp_3, J4 PWR_in, J5 SW_Fan_GND, J6 rs-485, J7 temp_4, J8 O2_sensor, J9 GND_conn, Q1 IRLS3036, U1 ATtiny3216-S, U2 AP63205WU, U3 AP2112K-3.3, U4 MCP1406-E/SN, U5 THVD1420D, U6 MCP6561x-LT

Commit message: checkpoint
Parts:
- R14: value 100k -> 10k
- R15: value 6.8k -> 2k
- R16: value 330k -> 100k
- U3: value AP2112K-3.3 -> AP2115M-3.3TRG1
Connections:
- net at R16.1, U6.1: now also U1.7 (PB4); no longer U1.9 (PB2)
- net at U1.4 (PA6): now also C15.2, R11.1, R9.2
- now unconnected: U1.8 (PB3)
Changed lines of the file:
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@@
 	)
 	(junction
+		(at 146.05 105.41)
+		(diameter 0)
+		(color 0 0 0 0)
+	)
+	(junction
 		(at 201.93 76.2)
 		(diameter 0)
@@
 	)
 	(junction
-		(at 187.96 156.21)
+		(at 44.45 158.75)
 		(diameter 0)
 		(color 0 0 0 0)
 	)
 	(junction
-		(at 44.45 158.75)
+		(at 66.04 163.83)
 		(diameter 0)
 		(color 0 0 0 0)
 	)
 	(junction
-		(at 66.04 163.83)
+		(at 134.62 44.45)
 		(diameter 0)
 		(color 0 0 0 0)
 	)
 	(junction
-		(at 134.62 44.45)
+		(at 187.96 143.51)
 		(diameter 0)
 		(color 0 0 0 0)
@@
 	)
 	(junction
-		(at 146.05 105.41)
-		(diameter 0)
-		(color 0 0 0 0)
-	)
-	(junction
 		(at 157.48 48.26)
 		(diameter 0)
@@
 	(wire
 		(pts
-			(xy 187.96 139.7) (xy 187.96 147.32)
+			(xy 187.96 139.7) (xy 187.96 143.51)
 		)
 		(stroke
@@
 	(wire
 		(pts
+			(xy 118.11 91.44) (xy 109.22 91.44)
+		)
+		(stroke
+			(width 0)
+			(type default)
+		)
+	)
+	(wire
+		(pts
 			(xy 115.57 166.37) (xy 115.57 187.96)
 		)
@@
 	(wire
 		(pts
-			(xy 187.96 156.21) (xy 187.96 158.75)
-		)
-		(stroke
-			(width 0)
-			(type default)
-		)
-	)
-	(wire
-		(pts
 			(xy 190.5 63.5) (xy 196.85 63.5)
 		)
@@
 	(wire
 		(pts
-			(xy 115.57 48.26) (xy 147.32 48.26)
+			(xy 187.96 143.51) (xy 187.96 147.32)
 		)
 		(stroke
@@
 	(wire
 		(pts
-			(xy 30.48 60.96) (xy 39.37 60.96)
+			(xy 115.57 48.26) (xy 147.32 48.26)
 		)
 		(stroke
@@
 	(wire
 		(pts
-			(xy 146.05 105.41) (xy 146.05 88.9)
+			(xy 30.48 60.96) (xy 39.37 60.96)
 		)
 		(stroke
@@
 	(wire
 		(pts
-			(xy 146.05 88.9) (xy 118.11 88.9)
-		)
-		(stroke
-			(width 0)
-			(type default)
-		)
-	)
-	(wire
-		(pts
 			(xy 58.42 148.59) (xy 58.42 149.86)
 		)
@@
 	(wire
 		(pts
-			(xy 109.22 86.36) (xy 118.11 86.36)
-		)
-		(stroke
-			(width 0)
-			(type default)
-		)
-	)
-	(wire
-		(pts
 			(xy 53.34 111.76) (xy 53.34 115.57)
 		)
@@
 	(wire
 		(pts
-			(xy 187.96 156.21) (xy 171.45 156.21)
-		)
-		(stroke
-			(width 0)
-			(type default)
-		)
-	)
-	(wire
-		(pts
 			(xy 119.38 34.29) (xy 115.57 34.29)
 		)
@@
 	(wire
 		(pts
-			(xy 171.45 156.21) (xy 171.45 166.37)
+			(xy 171.45 143.51) (xy 171.45 166.37)
 		)
 		(stroke
@@
 	(wire
 		(pts
-			(xy 109.22 86.36) (xy 109.22 148.59)
-		)
-		(stroke
-			(width 0)
-			(type default)
-		)
-	)
-	(wire
-		(pts
 			(xy 118.11 63.5) (xy 129.54 63.5)
 		)
@@
 	(wire
 		(pts
+			(xy 146.05 73.66) (xy 118.11 73.66)
+		)
+		(stroke
+			(width 0)
+			(type default)
+		)
+	)
+	(wire
+		(pts
 			(xy 45.72 74.93) (xy 45.72 60.96)
 		)
@@
 	(wire
 		(pts
+			(xy 146.05 105.41) (xy 146.05 73.66)
+		)
+		(stroke
+			(width 0)
+			(type default)
+		)
+	)
+	(wire
+		(pts
 			(xy 26.67 167.64) (xy 26.67 180.34)
 		)
@@
 	(wire
 		(pts
+			(xy 171.45 143.51) (xy 187.96 143.51)
+		)
+		(stroke
+			(width 0)
+			(type default)
+		)
+	)
+	(wire
+		(pts
 			(xy 134.62 66.04) (xy 118.11 66.04)
 		)
@@
 	(wire
 		(pts
-			(xy 187.96 147.32) (xy 187.96 156.21)
+			(xy 187.96 147.32) (xy 187.96 158.75)
 		)
 		(stroke
@@
 	(wire
 		(pts
+			(xy 109.22 91.44) (xy 109.22 148.59)
+		)
+		(stroke
+			(width 0)
+			(type default)
+		)
+	)
+	(wire
+		(pts
 			(xy 195.58 158.75) (xy 196.85 158.75)
 		)
@@
 	(wire
 		(pts
-			(xy 120.65 91.44) (xy 118.11 91.44)
-		)
-		(stroke
-			(width 0)
-			(type default)
-		)
-	)
-	(wire
-		(pts
 			(xy 157.48 59.69) (xy 172.72 59.69)
 		)
@@
 			)
 		)
-		(property "Value" "AP2112K-3.3"
+		(property "Value" "AP2115M-3.3TRG1"
 			(at 171.45 44.45 0)
 			(show_name no)
@@
 			)
 		)
-		(property "Value" "6.8k"
+		(property "Value" "2k"
 			(at 46.99 179.0699 0)
 			(show_name no)
@@
 			)
 		)
-		(property "Value" "100k"
+		(property "Value" "10k"
 			(at 46.99 170.1799 0)
 			(show_name no)
@@
 			)
 		)
-		(property "Value" "330k"
+		(property "Value" "100k"
 			(at 60.96 153.6699 0)
 			(show_name no)

Commit message: engine monitor code
Parts:
- R16: value 100k -> 47k
Connections:
- net at C17.2, D3.2 (A), D4.1 (K)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: no longer R16.2
- net at R14.2, R15.1, U6.4 (-): now also R16.2
Other:
- moved on the sheet: R16
Changed lines of the file:
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@@
 	)
 	(junction
+		(at 97.79 148.59)
+		(diameter 0)
+		(color 0 0 0 0)
+	)
+	(junction
 		(at 30.48 69.85)
 		(diameter 0)
@@
 	)
 	(junction
+		(at 72.39 163.83)
+		(diameter 0)
+		(color 0 0 0 0)
+	)
+	(junction
 		(at 187.96 168.91)
 		(diameter 0)
@@
 	)
 	(junction
-		(at 69.85 148.59)
-		(diameter 0)
-		(color 0 0 0 0)
-	)
-	(junction
 		(at 161.29 118.11)
 		(diameter 0)
@@
 	)
 	(junction
-		(at 66.04 163.83)
-		(diameter 0)
-		(color 0 0 0 0)
-	)
-	(junction
 		(at 134.62 44.45)
 		(diameter 0)
@@
 	(wire
 		(pts
+			(xy 97.79 163.83) (xy 72.39 163.83)
+		)
+		(stroke
+			(width 0)
+			(type default)
+		)
+	)
+	(wire
+		(pts
 			(xy 173.99 16.51) (xy 173.99 21.59)
 		)
@@
 	(wire
 		(pts
-			(xy 58.42 148.59) (xy 58.42 149.86)
+			(xy 97.79 148.59) (xy 97.79 152.4)
 		)
 		(stroke
@@
 	(wire
 		(pts
+			(xy 97.79 157.48) (xy 97.79 163.83)
+		)
+		(stroke
+			(width 0)
+			(type default)
+		)
+	)
+	(wire
+		(pts
 			(xy 130.81 133.35) (xy 130.81 134.62)
 		)
@@
 	(wire
 		(pts
-			(xy 58.42 163.83) (xy 66.04 163.83)
-		)
-		(stroke
-			(width 0)
-			(type default)
-		)
-	)
-	(wire
-		(pts
 			(xy 118.11 63.5) (xy 129.54 63.5)
 		)
@@
 	(wire
 		(pts
-			(xy 69.85 148.59) (xy 58.42 148.59)
+			(xy 97.79 148.59) (xy 69.85 148.59)
 		)
 		(stroke
@@
 	(wire
 		(pts
-			(xy 58.42 154.94) (xy 58.42 163.83)
-		)
-		(stroke
-			(width 0)
-			(type default)
-		)
-	)
-	(wire
-		(pts
 			(xy 157.48 124.46) (xy 157.48 125.73)
 		)
@@
 	(wire
 		(pts
-			(xy 109.22 148.59) (xy 69.85 148.59)
+			(xy 109.22 148.59) (xy 97.79 148.59)
 		)
 		(stroke
@@
 	(symbol
 		(lib_id "Device:R_Small_US")
-		(at 58.42 152.4 0)
+		(at 97.79 154.94 0)
 		(unit 1)
 		(body_style 1)
@@
 		(fields_autoplaced yes)
 		(property "Reference" "R16"
-			(at 60.96 151.1299 0)
+			(at 100.33 153.6699 0)
 			(show_name no)
 			(do_not_autoplace no)
@@
 			)
 		)
-		(property "Value" "100k"
-			(at 60.96 153.6699 0)
+		(property "Value" "47k"
+			(at 100.33 156.2099 0)
 			(show_name no)
 			(do_not_autoplace no)
@@
 		)
 		(property "Footprint" "Resistor_SMD:R_1206_3216Metric_Pad1.30x1.75mm_HandSolder"
-			(at 58.42 152.4 0)
+			(at 97.79 154.94 0)
 			(hide yes)
 			(show_name no)
@@
 		)
 		(property "Datasheet" ""
-			(at 58.42 152.4 0)
+			(at 97.79 154.94 0)
 			(hide yes)
 			(show_name no)
@@
 		)
 		(property "Description" "Resistor, small US symbol"
-			(at 58.42 152.4 0)
+			(at 97.79 154.94 0)
 			(hide yes)
 			(show_name no)
