File: display/display_pcb/display_pcb.kicad_sch (KiCad schematic)
At the start: 32 parts, among them J1 ESP32-S3-44-Pin, J2 4" TFT SPI DISPLAY, J3 Power_in, J4 RS-485_out, Q1 FDN340P, Q2 MMBT3904, U1 AP63205WU, U2 AP2115M-3.3TRG1, U3 THVD1420D

Commit message: PCB Updates
Parts:
- added C10: 22uF, Capacitor_SMD:C_1206_3216Metric_Pad1.33x1.80mm_HandSolder, symbol Device:C_Small_US
- added R11: 10k, Resistor_SMD:R_1206_3216Metric_Pad1.30x1.75mm_HandSolder, symbol Device:R_US
- added TH1: Thermistor_NTC_US, Resistor_SMD:R_1206_3216Metric_Pad1.30x1.75mm_HandSolder, symbol Device:Thermistor_NTC_US
- added TP1: 5V, TestPoint:TestPoint_Pad_2.5x2.5mm, symbol Connector:TestPoint
- added TP2: 3.3V, TestPoint:TestPoint_Pad_2.5x2.5mm, symbol Connector:TestPoint
- F1: footprint (none) -> Fuse:Fuseholder_Blade_Mini_Keystone_3568
- J1: footprint RF_Module:ESP32-C3-30pin-Alex -> Connector_PinHeader_2.54mm:PinHeader_1x22_P2.54mm_Vertical
- J2: footprint Connector_PinSocket_2.54mm:TFT-14pin-Alex -> Connector_PinHeader_2.54mm:PinHeader_1x14_P2.54mm_Vertical
- J3, J4: footprint (none) -> Connector:Alex_2pin_65thou
- L1: value L -> 4.7uH; footprint (none) -> Inductor_SMD:L_1008_2520Metric_Pad1.43x2.20mm_HandSolder
- R10, R8: value 100k -> 10k
- R2: value 5k -> 2k
- R3: value 10k -> 2k
- R4: value 100k -> 120
Connections:
- net GND: now also C5.1, C6.1, C7.1, C8.1, C9.1, D2.3 (common), U2.6 (GND), U2.7 (GND), U3.5 (GND), C10.2, TH1.2
- net 5V: now reaches C6.2, C9.2, J2.VCC (Pin_1), L1.1, Q1.2 (S), U2.5 (EN), U2.8 (VIN)
- net 5V: now also C1.1, C2.1, U1.1 (FB), R11.1, TP1.1; no longer R10.1
- net at Q2.3 (C), R7.1: no longer R10.2
- net at C3.1, D1.1 (K), F1.1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: now also C10.1
- net at Q2.1 (B), R9.1: no longer R8.1
- net at J2.CS (Pin_3): now also J1.14 (Pin_2), J2.T_CS
- net at J2.DC (Pin_5): now also J1.12 (Pin_4)
- net at J2.GND (Pin_2): now also J1.GND (3.3)
- net at J2.LED (Pin_8), Q1.3 (D): no longer C1.1, C2.1
- net at J2.MOSI (Pin_6): now also J1.11 (Pin_5), J2.T_DIN (Pin_12)
- net at J2.RST (Pin_4): now also J1.13 (Pin_3)
- net at J2.SCK (Pin_7): now also J1.10 (Pin_6), J2.T_CLK (Pin_10)
- net at J2.T_DO: now also J1.18 (Pin_5)
- net at J1.5 (Pin_11), R9.2: now also R8.1
- net at R1.1: now also J1.1 (Pin_12), R2.1
- net at R1.2: now also J1.GND (3.3)
- net at U3.1 (RO): now also J1.RX (Pin_13)
- net at U3.2 (~{RE}): now also J1.42 (Pin_10), U3.3 (DE)
- net at U3.4 (DI): now also J1.TX (36)
- net at U3.6 (A): now also D2.2 (A2), J4.1 (Pin_1), R4.2
- net at U3.7 (B): now also D2.1 (A1), J4.2 (Pin_2), R4.1
- net 3.3V: now reaches U3.8 (VCC)
- net 3.3V: now also C5.2, C7.2, C8.2, J1.3.3V (36), R2.2, R3.1, U2.1 (VOUT), TP2.1
- net at R3.2: now also J1.21 (Pin_4), TH1.1
- net at R5.1, R6.2: now also J1.2 (Pin_11)
- net at Q1.1 (G), R7.2: now also R11.2
Other:
- note added: "Supply voltage sensor"
- moved on the sheet: C1, C2, C5, C6, C7, C8, C9, D1, D2, F1, J4, Q1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
